File: CartePrincipale.brd (EAGLE design)
At the start: 182.9 x 125.7 mm, 99 parts

Commit message: ceci est un commit
Parts:
- moved 19 1.27 mm to (152.4, 118.1)
Routing:
- net GND: track 1025.3 -> 1072.5 mm
- net N$22: track 21.9 -> 22.4 mm

Commit message: ceci est un commit : le retour
Routing:
- net N$24: track 27.3 -> 26.2 mm
Changed lines of the file:
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@@
 <wire x1="181.61" y1="115.57" x2="182.88" y2="116.84" width="1.016" layer="16"/>
 <wire x1="182.88" y1="116.84" x2="182.88" y2="120.65" width="1.016" layer="16"/>
-<wire x1="182.88" y1="135.89" x2="193.04" y2="135.89" width="0.3048" layer="16"/>
-<wire x1="204.47" y1="148.59" x2="203.2" y2="148.59" width="0.3048" layer="16"/>
-<wire x1="203.2" y1="148.59" x2="201.93" y2="147.32" width="0.3048" layer="16"/>
-<wire x1="201.93" y1="147.32" x2="201.93" y2="137.16" width="0.3048" layer="16"/>
-<wire x1="201.93" y1="137.16" x2="200.66" y2="135.89" width="0.3048" layer="16"/>
-<wire x1="200.66" y1="135.89" x2="194.31" y2="135.89" width="0.3048" layer="16"/>
-<wire x1="194.31" y1="135.89" x2="193.0654" y2="135.89" width="0.3048" layer="16"/>
+<wire x1="182.88" y1="135.89" x2="193.04" y2="135.89" width="1.016" layer="16"/>
+<wire x1="204.47" y1="148.59" x2="203.2" y2="148.59" width="1.016" layer="16"/>
+<wire x1="203.2" y1="148.59" x2="201.93" y2="147.32" width="1.016" layer="16"/>
+<wire x1="201.93" y1="147.32" x2="201.93" y2="137.16" width="1.016" layer="16"/>
+<wire x1="201.93" y1="137.16" x2="200.66" y2="135.89" width="1.016" layer="16"/>
+<wire x1="200.66" y1="135.89" x2="194.31" y2="135.89" width="1.016" layer="16"/>
+<wire x1="194.31" y1="135.89" x2="193.0654" y2="135.89" width="1.016" layer="16"/>
 <wire x1="45.72" y1="128.27" x2="45.72" y2="133.35" width="3.81" layer="1"/>
 <wire x1="45.72" y1="133.35" x2="48.26" y2="135.89" width="3.81" layer="1"/>
@@
 <wire x1="194.98" y1="167.04" x2="195.58" y2="167.64" width="1.016" layer="16"/>
 <contactref element="JP1" pad="1"/>
-<wire x1="193.04" y1="138.43" x2="193.04" y2="137.16" width="0.3048" layer="16"/>
-<wire x1="193.04" y1="137.16" x2="194.31" y2="135.89" width="0.3048" layer="16"/>
+<wire x1="193.04" y1="138.43" x2="193.04" y2="137.16" width="1.016" layer="16"/>
+<wire x1="193.04" y1="137.16" x2="194.31" y2="135.89" width="1.016" layer="16"/>
 <wire x1="196.54" y1="127" x2="196.5" y2="127" width="1.016" layer="16"/>
 <wire x1="196.5" y1="127" x2="196.5" y2="113.03" width="1.016" layer="16"/>
@@
 <contactref element="3" pad="+"/>
 <contactref element="L5" pad="2"/>
-<wire x1="204.47" y1="146.05" x2="203.2" y2="144.78" width="0.3048" layer="16"/>
-<wire x1="203.2" y1="144.78" x2="203.2" y2="133.945" width="0.3048" layer="16"/>
-<wire x1="203.2" y1="133.945" x2="205.145" y2="132.08" width="0.3048" layer="16"/>
 <wire x1="204.47" y1="146.05" x2="207.01" y2="146.05" width="1.9304" layer="1"/>
 <wire x1="207.01" y1="146.05" x2="208.28" y2="147.32" width="1.9304" layer="1"/>
 <wire x1="208.28" y1="147.32" x2="208.28" y2="154.94" width="1.9304" layer="1"/>
+<wire x1="204.47" y1="146.05" x2="204.47" y2="132.755" width="0.254" layer="16"/>
+<wire x1="204.47" y1="132.755" x2="205.145" y2="132.08" width="0.254" layer="16"/>
 </signal>
 <signal name="9V1">

Commit message: Ceci est un commit : la menace de la loli
Routing:
- net GND: track 1072.5 -> 1064.6 mm
- net N$22: track 22.4 -> 23.2 mm

Commit message: Ceci est un commit : la revanche du 1A
Routing:
- net +5V: track 361.6 -> 364.2 mm
- net US4: track 164.1 -> 164.9 mm
- added copper zone on layer 1, net GND
- added copper zone on layer 16, net GND
Other:
- board size 182.9 x 125.7 mm -> 182.9 x 125.4 mm
