File: secondaire.brd (EAGLE design)
At the start: 54.6 x 54.6 mm, 22 parts

Commit message: Ceci est un commit : la revanche du 1A
Parts:
- moved C2 6.35 mm to (16.5, 31.8)
- moved L1 4.82 mm to (15.8, 12.2)
- moved C1 4.58 mm to (26.7, 11.4)
- moved R5 2.54 mm to (25.4, 44.5)
- moved R6 2.54 mm to (25.4, 40.6)
- moved U$1 2.54 mm to (35.6, 44.5)
Routing:
- net N$3: track 25.5 -> 34.3 mm
- net +12V: track 59.9 -> 64.0 mm
- net RX&TX: track 9.72 -> 13.7 mm
- net GND: track 166.6 -> 170.0 mm
- net +9V: track 17.6 -> 15.0 mm
- net N$20: track 5.61 -> 3.81 mm
Other:
- board size 54.6 x 54.6 mm -> 54.6 x 55.9 mm
- board text added: "+"
- board text added: "-"
- board text added: "12V"
- board text added: "5V"
- board text added: "A0"
- board text added: "AU"
- board text added: "C"
- board text added: "D:/INTech/intech_logo.bmp"
- board text added: "GND"
- board text added: "MOT"
- board text added: "NC"
- board text added: "NO"
